File: KiCad/HV servo drive v1/HV servo drive v1.kicad_sch (KiCad schematic)
At the start: 221 parts, among them J1 555153-1, J2 555153-1, J3 Conn_02x03_Odd_Even, J4 OSTYK51104030, J5 Conn_01x03_Female, J6 Conn_01x03_Female, J7 Conn_01x03_Female, M1 Fan_4pin, M2 Fan_4pin, Q1 C3M0075120K, Q2 C3M0075120K, Q3 C3M0075120K, Q4 C3M0075120K, Q5 C3M0075120K, Q6 C3M0075120K, SW1 SW_DIP_x04, U1 THVD1452DGSR, U10 LF2190NTR, U11 LF2190NTR, U12 LF2190NTR, U13 AMC1306M25DWVR, U14 AMC1306M25DWVR, U15 AMC1306M25DWVR, U2 ISO6721BQDRQ1, U3 ISO6721BQDRQ1, U4 ISO6721BQDRQ1, U5 STM32F413RGT6, U6 AP64060QWU-7, U7 CRE1S2412SC, U8 AP64060QWU-7, U9 AP64060QWU-7

Commit message: main update to v1.1 design
Parts:
- removed C1, C14, C15, C17, C2, C20, C21, C26, C28, C29, C3, C30, C31, C33, C34, C35, C36, C4, C5, C50, C51, C56, C59, C6, C61, C63, C68, C69, C7, C70: 0.1uf, Capacitor_SMD:C_0603_1608Metric, symbol Device:C
- removed C11, C25, C37, C38: .1uf, Capacitor_SMD:C_0603_1608Metric, symbol Device:C
- removed C12, C13, C40, C41, C47, C48, C49: 2.2uf, Capacitor_SMD:C_0603_1608Metric, symbol Device:C
- removed C16, C19, C42, C43, C44, C45, C52, C54, C57: 10uf, Capacitor_SMD:C_0805_2012Metric, symbol Device:C
- removed C18, C22, C23, C24, C27, C32, C39: 1uf, Capacitor_SMD:C_0603_1608Metric, symbol Device:C
- removed C46: ?, Capacitor_SMD:C_0805_2012Metric, symbol Device:C
- removed C53, C55, C58, C60, C62, C64: 22uf, Capacitor_SMD:C_0805_2012Metric, symbol Device:C
- removed C65, C66, C67: 2.2, Capacitor_SMD:C_0603_1608Metric, symbol Device:C
- removed C71, C72, C73: C, Capacitor_SMD:C_0603_1608Metric, symbol Device:C
- removed C8, C9: 40uf, hv servo drive footprints:BUS CAP1, symbol Device:C
- removed D1, D2: D_TVS_Dual_AAC, Package_TO_SOT_SMD:SOT-23, symbol Device:D_TVS_Dual_AAC
- removed D10, D11, D12, D13, D14, D15, D7, D8, D9: D_Dual_Series_ACK, Package_TO_SOT_SMD:SOT-23, symbol Device:D_Dual_Series_AKC
- removed D16, D17, D18: D, hv servo drive footprints:CR_ES3J_ONS, symbol Device:D
- removed D19, D20, D21: 1N751A, Diode_SMD:D_SOD-123, symbol Device:D_Zener
- removed D3, D4, D5, D6: LED, LED_SMD:LED_0603_1608Metric, symbol Device:LED
- removed H1, H2: MountingHole_Pad, MountingHole:MountingHole_3.2mm_M3_DIN965_Pad_TopBottom, symbol Mechanical:MountingHole_Pad
- removed H3, H4: MountingHole, MountingHole:MountingHole_3.2mm_M3_DIN965_Pad_TopBottom, symbol Mechanical:MountingHole
- removed J1, J2: 555153-1, hv servo drive footprints:CONN_555153-1_TYC, symbol 2023-05-31_00-30-22:555153-1
- removed J3: Conn_02x03_Odd_Even, Connector_PinHeader_2.54mm:PinHeader_2x03_P2.54mm_Vertical, symbol Connector_Generic:Conn_02x03_Odd_Even
- removed J4: OSTYK51104030, hv servo drive footprints:CONN04_OSTYK51_40X16P1_OST, symbol 2023-05-17_01-08-34:OSTYK51104030
- removed J5, J6, J7: Conn_01x03_Female, Connector_Wire:SolderWire-0.5sqmm_1x03_P4.6mm_D0.9mm_OD2.1mm, symbol Connector:Conn_01x03_Female
- removed L1, L2, L3: 10uH, Inductor_SMD:L_1008_2520Metric, symbol Device:L
- removed L4: ?, Inductor_SMD:L_1008_2520Metric, symbol Device:L
- removed M1, M2: Fan_4pin, Connector_PinHeader_2.54mm:PinHeader_1x04_P2.54mm_Vertical, symbol Motor:Fan_4pin
- removed NT1, NT2, NT3: NetTie_2, NetTie:NetTie-2_SMD_Pad0.5mm, symbol Device:NetTie_2
- removed Q1, Q2, Q3, Q4, Q5, Q6: C3M0075120K, hv servo drive footprints:TO-247-4_Horizontal_TabUp, symbol SiC FET:C3M0075120K
- removed R1, R2, R3, R4: 10, Resistor_SMD:R_0603_1608Metric, symbol Device:R
- removed R10, R15, R18, R19, R20, R21, R22, R23, R24, R37, R46, R7, R8, R9: 10k, Resistor_SMD:R_0603_1608Metric, symbol Device:R
- removed R11, R12, R13, R14: 1k, Resistor_SMD:R_0603_1608Metric, symbol Device:R
- removed R16, R31: 50k, Resistor_SMD:R_0603_1608Metric, symbol Device:R
- removed R17, R26, R28, R30, R32, R39, R41, R43, R45: 5k, Resistor_SMD:R_0603_1608Metric, symbol Device:R
- removed R25, R27, R29, R38, R40, R42, R44: 1M, Resistor_THT:R_Axial_DIN0309_L9.0mm_D3.2mm_P12.70mm_Horizontal, symbol Device:R
- removed R33: 69.8k, Resistor_SMD:R_0603_1608Metric, symbol Device:R
- removed R34, R36, R6: 22.1k, Resistor_SMD:R_0603_1608Metric, symbol Device:R
- removed R35: 475k, Resistor_SMD:R_0603_1608Metric, symbol Device:R
- removed R47, R48, R49: 1, Resistor_SMD:R_0805_2012Metric, symbol Device:R
- removed R5: 115k, Resistor_SMD:R_0603_1608Metric, symbol Device:R
- removed R50, R51, R56: 800, Resistor_SMD:R_0805_2012Metric, symbol Device:R
- removed R52, R53, R54, R55, R57, R58: 3, Resistor_SMD:R_1206_3216Metric, symbol Device:R
- removed R59, R60, R62, R64, R66, R67: R, Resistor_SMD:R_0603_1608Metric, symbol Device:R
- removed R61, R63, R65: .005, hv servo drive footprints:RES_HCSM2818_STP, symbol Device:R
- removed SW1: SW_DIP_x04, Package_DIP:DIP-8_W7.62mm, symbol Switch:SW_DIP_x04
- removed TH1, TH2, TH3: Thermistor, Connector_PinHeader_2.54mm:PinHeader_1x02_P2.54mm_Vertical, symbol Device:Thermistor
- removed TP1, TP10, TP11, TP12, TP13, TP14, TP15, TP16, TP2, TP3, TP4, TP5, TP6, TP7, TP8, TP9: TestPoint, hv servo drive footprints:TestPoint_Pad_3.1x1.6mm, symbol Connector:TestPoint
- removed U1: THVD1452DGSR, hv servo drive footprints:DGS0010A_N, symbol 2023-05-31_01-39-08:THVD1452DGSR
- removed U10, U11, U12: LF2190NTR, hv servo drive footprints:SOICN-8_LTF, symbol 2023-05-15_23-01-16:LF2190NTR
- removed U13, U14, U15: AMC1306M25DWVR, hv servo drive footprints:DWV0008A, symbol 2023-05-15_23-02-57:AMC1306M25DWVR
- removed U2, U3, U4: ISO6721BQDRQ1, hv servo drive footprints:SOICN-8_LTF, symbol 2023-05-31_00-34-52:ISO6721BQDRQ1
- removed U5: STM32F413RGT6, hv servo drive footprints:LQFP64-10x10mm, symbol 2023-05-15_23-02-32:STM32F413RGT6
- removed U6, U8, U9: AP64060QWU-7, hv servo drive footprints:IC6_AP64060QWU-7_DIO, symbol 2023-05-31_19-45-09:AP64060QWU-7
- removed U7: CRE1S2412SC, hv servo drive footprints:24v isolated converter, symbol 2023-05-15_23-02-57:DC-DC_converter
Other:
- added sheet ADC Sense (adc sense.kicad_sch)
- added sheet Controller Interface (controller interface.kicad_sch)
- added sheet Gate Supplies (gate supplies.kicad_sch)
- added sheet MCU (mcu.kicad_sch)
- added sheet Mounting (mounting.kicad_sch)
- added sheet Phase Bridges (phase bridges.kicad_sch)
- added sheet Power Connectors (power connectors.kicad_sch)
- added sheet STO (sto.kicad_sch)
- added sheet User IO (user io.kicad_sch)
