File: KiCad/HV servo drive v1/HV servo drive v1.kicad_pcb (KiCad board)
At the start: 4 copper layers, 99.8 x 99.3 mm, 221 parts, among them J1 555153-1, J2 555153-1, J3 Conn_02x03_Odd_Even, J4 OSTYK51104030, J5 Conn_01x03_Female, J6 Conn_01x03_Female, J7 Conn_01x03_Female, M1 Fan_4pin, M2 Fan_4pin, Q1 C3M0075120K, Q2 C3M0075120K, Q3 C3M0075120K, Q4 C3M0075120K, Q5 C3M0075120K, Q6 C3M0075120K, SW1 SW_DIP_x04, U1 THVD1452DGSR, U10 LF2190NTR, U11 LF2190NTR, U12 LF2190NTR, U13 AMC1306M25DWVR, U14 AMC1306M25DWVR, U15 AMC1306M25DWVR, U2 ISO6721BQDRQ1, U3 ISO6721BQDRQ1, U4 ISO6721BQDRQ1, U5 STM32F413RGT6, U6 AP64060QWU-7, U7 CRE1S2412SC, U8 AP64060QWU-7, U9 AP64060QWU-7

Commit message: main update to v1.1 design
Parts:
- removed D11, D7: D_Dual_Series_ACK, Package_TO_SOT_SMD:SOT-23
- removed H2: MountingHole_Pad, MountingHole:MountingHole_3.2mm_M3_DIN965_Pad_TopBottom
- removed J1, J2: 555153-1, hv servo drive footprints:CONN_555153-1_TYC
- removed J4: OSTYK51104030, hv servo drive footprints:CONN04_OSTYK51_40X16P1_OST
- removed NT1, NT2, NT3: NetTie_2, NetTie:NetTie-2_SMD_Pad0.5mm
- removed R15, R7, R8, R9: 10k, Resistor_SMD:R_0603_1608Metric
- removed R16, R31: 50k, Resistor_SMD:R_0603_1608Metric
- removed R17, R32: 5k, Resistor_SMD:R_0603_1608Metric
- added C10: 10uf, Capacitor_SMD:C_0805_2012Metric, F.Cu at (408.4, 120.0)
- added C100: 10uf, Capacitor_SMD:C_0805_2012Metric, F.Cu at (398.8, 56.0)
- added C101: 10uf, Capacitor_SMD:C_0805_2012Metric, F.Cu at (405.5, 72.0)
- added C102: 10uf, Capacitor_SMD:C_0805_2012Metric, F.Cu at (402.8, 76.3)
- added C103: 10uf, Capacitor_SMD:C_0805_2012Metric, F.Cu at (402.8, 87.5)
- added C104: 10uf, Capacitor_SMD:C_0805_2012Metric, F.Cu at (392.8, 83.5)
- added C105: 10uf, Capacitor_SMD:C_0805_2012Metric, F.Cu at (388.8, 86.5)
- added C106: 10uf, Capacitor_SMD:C_0805_2012Metric, F.Cu at (391.5, 99.5)
- added C107: 0.1uf, Capacitor_SMD:C_0603_1608Metric, F.Cu at (338.8, 97.0)
- added C108: .1uf, Capacitor_SMD:C_2220_5650Metric, F.Cu at (382.4, 120.6)
- added C109: .1uf, Capacitor_SMD:C_2220_5650Metric, F.Cu at (382.4, 159.2)
- added C110: .1uf, Capacitor_SMD:C_2220_5650Metric, F.Cu at (382.4, 198.0)
- added C74: 10uf, Capacitor_SMD:C_0805_2012Metric, F.Cu at (403.6, 111.8)
- added C75: 0.1uf, Capacitor_SMD:C_0603_1608Metric, F.Cu at (407.2, 114.5)
- added C76: 0.1uf, Capacitor_SMD:C_0603_1608Metric, F.Cu at (405.7, 111.9)
- added C77: 10uf, Capacitor_SMD:C_0805_2012Metric, F.Cu at (410.0, 200.2)
- added C78: 10uf, Capacitor_SMD:C_0805_2012Metric, F.Cu at (408.3, 197.2)
- added C79: 0.1uf, Capacitor_SMD:C_0603_1608Metric, F.Cu at (411.3, 198.7)
- added C80: 0.1uf, Capacitor_SMD:C_0603_1608Metric, F.Cu at (417.9, 112.8)
- added C81: 0.1uf, Capacitor_SMD:C_0603_1608Metric, F.Cu at (409.8, 196.0)
- added C82: 10uf, Capacitor_SMD:C_0805_2012Metric, F.Cu at (405.3, 192.0)
- added C83: 10uf, Capacitor_SMD:C_0805_2012Metric, F.Cu at (403.5, 189.0)
- added C84: 0.1uf, Capacitor_SMD:C_0603_1608Metric, F.Cu at (407.2, 191.8)
- added C85: 0.1uf, Capacitor_SMD:C_0603_1608Metric, F.Cu at (405.7, 189.2)
- added C86: 2.2, Capacitor_SMD:C_0603_1608Metric, F.Cu at (403.4, 180.2)
- added C87: 0.1uf, Capacitor_SMD:C_0603_1608Metric, F.Cu at (405.1, 180.2)
- added C88: C, Capacitor_SMD:C_0603_1608Metric, F.Cu at (402.6, 183.5)
- added C89: 0.1uf, Capacitor_SMD:C_0603_1608Metric, F.Cu at (421.5, 95.0)
- added C90: 10uf, Capacitor_SMD:C_0805_2012Metric, F.Cu at (355.8, 59.0)
- added C91: 10uf, Capacitor_SMD:C_0805_2012Metric, F.Cu at (355.8, 65.8)
- added C92: 10uf, Capacitor_SMD:C_0805_2012Metric, F.Cu at (369.8, 55.0)
- added C93: 10uf, Capacitor_SMD:C_0805_2012Metric, F.Cu at (380.8, 58.6)
- added C94: 10uf, Capacitor_SMD:C_0805_2012Metric, F.Cu at (355.8, 57.0)
- added C95: 10uf, Capacitor_SMD:C_0805_2012Metric, F.Cu at (355.8, 63.8)
- added C96: 0.1uf, Capacitor_SMD:C_0603_1608Metric, F.Cu at (360.6, 92.2)
- added C97: 10uf, Capacitor_SMD:C_0805_2012Metric, F.Cu at (356.3, 74.5)
- added C98: 10uf, Capacitor_SMD:C_0805_2012Metric, F.Cu at (347.0, 74.5)
- added C99: 0.1uf, Capacitor_SMD:C_0603_1608Metric, F.Cu at (348.2, 93.5)
- added D22: D, Diode_SMD:D_SMB, F.Cu at (410.9, 134.9)
- added D23: D, Diode_SMD:D_SMB, F.Cu at (410.8, 212.2)
- added D24: BZT52C5V1, Diode_SMD:D_SOD-123, F.Cu at (399.9, 180.3)
- added D25: BZT52C5V1, Diode_SMD:D_SOD-123, F.Cu at (358.8, 74.2)
- added D26: D_Dual_Series_ACK, Package_TO_SOT_SMD:SOT-23, F.Cu at (353.3, 74.5)
- added D27: D_Dual_Series_ACK, Package_TO_SOT_SMD:SOT-23, F.Cu at (344.0, 74.5)
- added D28: BZT52C5V1, Diode_SMD:D_SOD-123, F.Cu at (349.5, 74.2)
- added D29: D_Dual_Series_ACK, Package_TO_SOT_SMD:SOT-23, F.Cu at (332.3, 76.9)
- added D30: BZT52C5V1, Diode_SMD:D_SOD-123, F.Cu at (332.0, 73.6)
- added F1: Polyfuse, Fuse:Fuse_1206_3216Metric, F.Cu at (317.0, 82.0)
- added F2: Polyfuse, Fuse:Fuse_1206_3216Metric, F.Cu at (317.0, 74.0)
- added H10: MountingHole, footprints:MountingHole_3.2mm_M3_Pad_TopBottom_LargeIsolation, F.Cu at (444.0, 246.0)
- added H12: MountingHole, footprints:MountingHole_3.2mm_M3_Pad_TopBottom_LargeIsolation, F.Cu at (315.0, 155.0)
- added H13: MountingHole, footprints:MountingHole_3.2mm_M3_Pad_TopBottom_LargeIsolation, F.Cu at (315.0, 197.0)
- added H14: MountingHole, footprints:MountingHole_3.2mm_M3_Pad_TopBottom_LargeIsolation, F.Cu at (345.0, 246.0)
- added H6: MountingHole, footprints:MountingHole_3.2mm_M3_Pad_TopBottom_LargeIsolation, F.Cu at (444.0, 98.0)
- added H7: MountingHole, footprints:MountingHole_3.2mm_M3_Pad_TopBottom_LargeIsolation, F.Cu at (444.0, 214.0)
- added H8: MountingHole, footprints:MountingHole_3.2mm_M3_Pad_TopBottom_LargeIsolation, F.Cu at (374.0, 181.0)
- added H9: MountingHole, footprints:MountingHole_3.2mm_M3_Pad_TopBottom_LargeIsolation, F.Cu at (444.0, 57.0)
- added J10: DC BUS J2, Connector_Molex:Molex_Mega-Fit_76825-0004_2x02_P5.70mm_Horizontal, B.Cu at (322.8, 140.7)
- added J8: 8P8C_LED_Shielded_x2, footprints:RJ45_E5908-0T0343-L, B.Cu at (316.4, 61.0)
- added J9: Conn_02x03_Top_Bottom, Connector_Molex:Molex_Mini-Fit_Jr_5569-06A2_2x03_P4.20mm_Horizontal, B.Cu at (320.8, 73.8)
- added L10: 10uH, Inductor_SMD:L_1008_2520Metric, F.Cu at (381.5, 86.2)
- added L11: 10uH, Inductor_SMD:L_0603_1608Metric, F.Cu at (405.6, 146.2)
- added L12: 10uH, Inductor_SMD:L_0603_1608Metric, F.Cu at (405.5, 186.6)
- added L13: 10uH, Inductor_SMD:L_0603_1608Metric, F.Cu at (403.9, 194.4)
- added L14: 10uH, Inductor_SMD:L_0603_1608Metric, F.Cu at (405.5, 185.0)
- added L15: 10uH, Inductor_SMD:L_1008_2520Metric, F.Cu at (408.8, 95.8)
- added L16: 10uH, Inductor_SMD:L_1008_2520Metric, F.Cu at (321.2, 54.5)
- added L17: 10uH, Inductor_SMD:L_1008_2520Metric, F.Cu at (317.0, 59.2)
- added L5: 10uH, Inductor_SMD:L_1008_2520Metric, F.Cu at (384.5, 55.2)
- added L6: 10uH, Inductor_SMD:L_1008_2520Metric, F.Cu at (402.8, 72.0)
- added L7: 10uH, Inductor_SMD:L_1008_2520Metric, F.Cu at (392.8, 86.2)
- added L8: 10uH, Inductor_SMD:L_0603_1608Metric, F.Cu at (405.6, 147.8)
- added L9: 10uH, Inductor_SMD:L_0603_1608Metric, F.Cu at (403.9, 155.7)
- added Q8: PMOS, Package_SO:SOIC-8_3.9x4.9mm_P1.27mm, F.Cu at (338.3, 75.9)
- added R68: 1, Resistor_SMD:R_0805_2012Metric, F.Cu at (405.9, 135.4)
- added R69: 1K, Resistor_SMD:R_0603_1608Metric, F.Cu at (335.0, 80.6)
- added R70: 10K, Resistor_SMD:R_0603_1608Metric, F.Cu at (339.8, 79.6)
- added R71: 1k, Resistor_SMD:R_0603_1608Metric, F.Cu at (356.8, 78.5)
- added R72: 1K, Resistor_SMD:R_0603_1608Metric, F.Cu at (354.8, 78.5)
- added R73: 1K, Resistor_SMD:R_0603_1608Metric, F.Cu at (353.0, 78.5)
- added R74: 1K, Resistor_SMD:R_0603_1608Metric, F.Cu at (367.5, 80.0)
- added R75: 10K, Resistor_SMD:R_0603_1608Metric, F.Cu at (408.0, 77.8)
- added R76: 10K, Resistor_SMD:R_0603_1608Metric, F.Cu at (408.0, 74.5)
- added R77: 1K, Resistor_SMD:R_0603_1608Metric, F.Cu at (343.8, 78.5)
- added R78: 1K, Resistor_SMD:R_0603_1608Metric, F.Cu at (345.5, 78.5)
- added R79: 1k, Resistor_SMD:R_0603_1608Metric, F.Cu at (349.3, 78.5)
- added R80: 10K, Resistor_SMD:R_0603_1608Metric, F.Cu at (438.0, 63.0)
- added R81: 10K, Resistor_SMD:R_0603_1608Metric, F.Cu at (438.0, 64.5)
- added R82: 1K, Resistor_SMD:R_0603_1608Metric, F.Cu at (438.0, 66.0)
- added R83: 1k, Resistor_SMD:R_0603_1608Metric, F.Cu at (347.5, 78.5)
- added R84: 1k, Resistor_SMD:R_0603_1608Metric, F.Cu at (358.5, 78.5)
- added R85: 220, Resistor_SMD:R_0603_1608Metric, F.Cu at (335.0, 92.6)
- added R86: 220, Resistor_SMD:R_0603_1608Metric, F.Cu at (331.5, 92.6)
- added R87: 10k, Resistor_SMD:R_0603_1608Metric, F.Cu at (340.0, 101.0)
- added R88: 10k, Resistor_SMD:R_0603_1608Metric, F.Cu at (342.8, 102.5)
- added R89: 10k, Resistor_SMD:R_0603_1608Metric, F.Cu at (329.5, 93.8)
- added R90: 120, Resistor_SMD:R_0603_1608Metric, F.Cu at (338.5, 64.5)
- added R91: 120, Resistor_SMD:R_0603_1608Metric, F.Cu at (334.5, 66.0)
- added SW2: TERM RES, Package_DIP:DIP-4_W7.62mm, B.Cu at (339.5, 66.8)
- added TP17: TestPoint, footprints:TestPoint_Pad_3.1x1.6mm, F.Cu at (422.5, 189.0)
- added TP22: TestPoint, footprints:TestPoint_Pad_3.1x1.6mm, F.Cu at (357.2, 95.8)
- added TP23: TestPoint, footprints:TestPoint_Pad_3.1x1.6mm, F.Cu at (352.5, 95.8)
- added TP24: TestPoint, footprints:TestPoint_Pad_3.1x1.6mm, F.Cu at (342.5, 95.8)
- added U16: 6N137, footprints:6N137S_LTO, F.Cu at (354.8, 86.6)
- added U17: 6N137, footprints:6N137S_LTO, F.Cu at (343.5, 86.6)
- added U18: FODM217A, Package_SO:SOP-4_4.4x2.6mm_P1.27mm, F.Cu at (332.3, 86.6)
- added U19: FODM217A, Package_SO:SOP-4_4.4x2.6mm_P1.27mm, F.Cu at (335.8, 86.6)
- added U20: WRF0505S-3WR2, footprints:F0505S-2WR3, B.Cu at (399.7, 74.9)
- added U21: B0505MT-1WR4, footprints:B05xxMT-1WR4_MNS, F.Cu at (379.1, 93.0)
- added U22: PL133-37TC, Package_TO_SOT_SMD:SOT-23-6, F.Cu at (424.0, 95.0)
- added U23: THVD1552, Package_SO:SOIC-14_3.9x8.7mm_P1.27mm, F.Cu at (345.5, 59.0)
- C1, C11, C13, C16, C19, C41, C42, C43, C44, D1, D2, L1, R1, R13, R14, R2, R24, R3, R37, R4, R46, R5, R6: moved to F.Cu
- C18, C23, C24: value 1uf -> 10uf; footprint Capacitor_SMD:C_0603_1608Metric -> Capacitor_SMD:C_0805_2012Metric
- C22: value 1uf -> 10uf; footprint Capacitor_SMD:C_0603_1608Metric -> Capacitor_SMD:C_0805_2012Metric; moved to F.Cu
- C26: value 0.1uf -> 220pf; moved to F.Cu
- C27, C32, C39: value 1uf -> 2.2uf; moved to F.Cu
- C31: value 0.1uf -> 220pf; footprint Capacitor_SMD:C_0603_1608Metric -> Capacitor_THT:C_Disc_D7.5mm_W5.0mm_P10.00mm
- C37: value .1uf -> 10uf; footprint Capacitor_SMD:C_0603_1608Metric -> Capacitor_SMD:C_0805_2012Metric; moved to F.Cu
- C38: value .1uf -> 2.2uf; moved to F.Cu
- C40: value 2.2uf -> 10uf; footprint Capacitor_SMD:C_0603_1608Metric -> Capacitor_SMD:C_0805_2012Metric; moved to F.Cu
- C45: value 10uf -> 0.1uf; footprint Capacitor_SMD:C_0805_2012Metric -> Capacitor_SMD:C_0603_1608Metric; moved to F.Cu
- C46: value ? -> 10uf; moved to F.Cu
- C47: value 2.2uf -> 10uf; footprint Capacitor_SMD:C_0603_1608Metric -> Capacitor_SMD:C_0805_2012Metric
- C48, C49: value 2.2uf -> 470uf; footprint Capacitor_SMD:C_0603_1608Metric -> Capacitor_THT:CP_Radial_D30.0mm_P10.00mm_SnapIn
- C53, C58, C62: value 22uf -> 10uf
- C55, C60: value 22uf -> 0.1uf; footprint Capacitor_SMD:C_0805_2012Metric -> Capacitor_SMD:C_0603_1608Metric
- C57: value 10uf -> 0.1uf; footprint Capacitor_SMD:C_0805_2012Metric -> Capacitor_SMD:C_0603_1608Metric
- C59, C70: value 0.1uf -> 10uf; footprint Capacitor_SMD:C_0603_1608Metric -> Capacitor_SMD:C_0805_2012Metric
- C64: value 22uf -> 2.2; footprint Capacitor_SMD:C_0805_2012Metric -> Capacitor_SMD:C_0603_1608Metric
- C65: value 2.2 -> 0.1uf
- C67: value 2.2 -> C
- C71: value C -> 10uf; footprint Capacitor_SMD:C_0603_1608Metric -> Capacitor_SMD:C_0805_2012Metric
- C73: value C -> 0.1uf
- C8, C9: footprint hv servo drive footprints:BUS CAP1 -> footprints:BUS CAP1
- D16, D17, D18: footprint hv servo drive footprints:CR_ES3J_ONS -> Diode_SMD:D_SMB
- D19, D20: value 1N751A -> BZT52C5V1
- D21: value 1N751A -> D; footprint Diode_SMD:D_SOD-123 -> Diode_SMD:D_SMB
- H1: value MountingHole_Pad -> MountingHole; footprint MountingHole:MountingHole_3.2mm_M3_DIN965_Pad_TopBottom -> footprints:MountingHole_3.2mm_M3_Pad_TopBottom_LargeIsolation
- H3, H4: footprint MountingHole:MountingHole_3.2mm_M3_DIN965_Pad_TopBottom -> footprints:MountingHole_3.2mm_M3_Pad_TopBottom_LargeIsolation
- J3: value Conn_02x03_Odd_Even -> PROG; moved to B.Cu
- J5: value Conn_01x03_Female -> MOTOR; footprint Connector_Wire:SolderWire-0.5sqmm_1x03_P4.6mm_D0.9mm_OD2.1mm -> Connector_Molex:Molex_Mega-Fit_76825-0008_2x04_P5.70mm_Horizontal; moved to B.Cu
- J6: value Conn_01x03_Female -> PFC SENSE; footprint Connector_Wire:SolderWire-0.5sqmm_1x03_P4.6mm_D0.9mm_OD2.1mm -> Connector_Molex:Molex_Mini-Fit_Jr_5569-04A2_2x02_P4.20mm_Horizontal
- J7: value Conn_01x03_Female -> DC BUS J1; footprint Connector_Wire:SolderWire-0.5sqmm_1x03_P4.6mm_D0.9mm_OD2.1mm -> Connector_Molex:Molex_Mega-Fit_76825-0004_2x02_P5.70mm_Horizontal; moved to B.Cu
- L2, L3: footprint Inductor_SMD:L_1008_2520Metric -> Inductor_SMD:L_0603_1608Metric; moved to F.Cu
- L4: value ? -> 10uH; footprint Inductor_SMD:L_1008_2520Metric -> Inductor_SMD:L_0603_1608Metric; moved to F.Cu
- M1, M2: footprint Connector_PinHeader_2.54mm:PinHeader_1x04_P2.54mm_Vertical -> Connector_Molex:Molex_SPOX_5267-04A_1x04_P2.50mm_Vertical; moved to B.Cu
- Q1, Q2, Q3, Q4, Q5, Q6: footprint hv servo drive footprints:TO-247-4_Horizontal_TabUp -> footprints:TO-247-4_Horizontal_TabUp
- R33: value 69.8k -> 1; footprint Resistor_SMD:R_0603_1608Metric -> Resistor_SMD:R_0805_2012Metric; moved to F.Cu
- R34: value 22.1k -> 1; footprint Resistor_SMD:R_0603_1608Metric -> Resistor_SMD:R_0805_2012Metric; moved to F.Cu
- R35: value 475k -> 800; footprint Resistor_SMD:R_0603_1608Metric -> Resistor_SMD:R_0805_2012Metric; moved to F.Cu
- R36: value 22.1k -> 10; footprint Resistor_SMD:R_0603_1608Metric -> Resistor_SMD:R_1206_3216Metric; moved to F.Cu
- R47: value 1 -> 10; footprint Resistor_SMD:R_0805_2012Metric -> Resistor_SMD:R_1206_3216Metric
- R49: value 1 -> R; footprint Resistor_SMD:R_0805_2012Metric -> Resistor_SMD:R_0603_1608Metric
- R50: value 800 -> .005; footprint Resistor_SMD:R_0805_2012Metric -> footprints:RES_HCSM2818_STP
- R52: value 3 -> R; footprint Resistor_SMD:R_1206_3216Metric -> Resistor_SMD:R_0603_1608Metric
- R53: value 3 -> 1; footprint Resistor_SMD:R_1206_3216Metric -> Resistor_SMD:R_0805_2012Metric
- R54, R55, R58: value 3 -> 10
- R56: value 800 -> 1
- R57: value 3 -> 800; footprint Resistor_SMD:R_1206_3216Metric -> Resistor_SMD:R_0805_2012Metric
- R59: value R -> 10; footprint Resistor_SMD:R_0603_1608Metric -> Resistor_SMD:R_1206_3216Metric
- R61: value .005 -> R; footprint hv servo drive footprints:RES_HCSM2818_STP -> Resistor_SMD:R_0603_1608Metric; moved to F.Cu
- R62: value R -> .005; footprint Resistor_SMD:R_0603_1608Metric -> footprints:RES_HCSM2818_STP
- R63: footprint hv servo drive footprints:RES_HCSM2818_STP -> footprints:RES_HCSM2818_STP; moved to F.Cu
- R65: value .005 -> 10K; footprint hv servo drive footprints:RES_HCSM2818_STP -> Resistor_SMD:R_0603_1608Metric; moved to F.Cu
- R67: value R -> 1K
- SW1: moved to B.Cu
- TH3: footprint Connector_PinHeader_2.54mm:PinHeader_1x02_P2.54mm_Vertical -> Resistor_SMD:R_0603_1608Metric
- TP1, TP10, TP11, TP12, TP13, TP14, TP15, TP16, TP2, TP3, TP4, TP5, TP6, TP7, TP8, TP9: footprint hv servo drive footprints:TestPoint_Pad_3.1x1.6mm -> footprints:TestPoint_Pad_3.1x1.6mm
- U1: value THVD1452DGSR -> TCA9555PWR; footprint hv servo drive footprints:DGS0010A_N -> Package_SO:TSSOP-24_4.4x7.8mm_P0.65mm; moved to F.Cu
- U10, U11: value LF2190NTR -> 2EDF9275FXUMA1; footprint hv servo drive footprints:SOICN-8_LTF -> footprints:PG-DSO-16-11
- U12: value LF2190NTR -> AMC1306M25DWVR; footprint hv servo drive footprints:SOICN-8_LTF -> footprints:DWV0008A
- U13: value AMC1306M25DWVR -> 2EDF9275FXUMA1; footprint hv servo drive footprints:DWV0008A -> footprints:PG-DSO-16-11
- U14, U15: footprint hv servo drive footprints:DWV0008A -> footprints:DWV0008A
- U2, U3, U4: footprint hv servo drive footprints:SOICN-8_LTF -> footprints:SOICN-8_LTF
- U5: footprint hv servo drive footprints:LQFP64-10x10mm -> footprints:LQFP64-10x10mm
- U6: footprint hv servo drive footprints:IC6_AP64060QWU-7_DIO -> footprints:IC6_AP64060QWU-7_DIO; moved to F.Cu
- U7: value CRE1S2412SC -> WRF0505S-3WR2; footprint hv servo drive footprints:24v isolated converter -> footprints:F0505S-2WR3; moved to B.Cu
- U8: value AP64060QWU-7 -> B0505MT-1WR4; footprint hv servo drive footprints:IC6_AP64060QWU-7_DIO -> footprints:B05xxMT-1WR4_MNS; moved to F.Cu
- U9: value AP64060QWU-7 -> AP2127K-3.3; footprint hv servo drive footprints:IC6_AP64060QWU-7_DIO -> Package_TO_SOT_SMD:SOT-23-5; moved to F.Cu
- moved H4 340.4 mm to (444.0, 157.0)
- moved C24 321.6 mm to (430.8, 197.7)
- moved TP13 311.0 mm to (422.5, 154.2), turned to 0 degrees
- moved U9 310.5 mm to (412.0, 57.6), turned to 0 degrees
- moved C38 309.9 mm to (408.7, 58.0), turned to 90 degrees
- moved R10 309.9 mm to (429.8, 60.2), turned to 0 degrees
- moved C45 308.7 mm to (417.9, 151.3), turned to 120 degrees
- moved C41 307.2 mm to (410.7, 55.0), turned to 180 degrees
- moved R35 303.9 mm to (411.4, 164.7), turned to 0 degrees
- moved R34 302.0 mm to (405.9, 173.9), turned to 90 degrees
- moved TP2 301.8 mm to (404.0, 55.8)
- moved R36 299.6 mm to (404.1, 164.6), turned to -150 degrees
- moved L3 299.6 mm to (405.6, 107.8), turned to 0 degrees
- moved U5 299.2 mm to (428.0, 72.0)
- moved C14 299.1 mm to (425.1, 79.6)
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Connections:
- C1 pad 1: +5V -> 5v_ISO
- C16 pad 1: +5V -> 5v_ISO
- C18 pad 1: 24V_ISO -> 5v_ISO
- C19 pad 1: +5V -> 5v_ISO
- C2 pad 1: +5V -> 5v_ISO
- C23 pad 1: +24V -> Net-(U7-VIN)
- C23 pad 2: GND2 -> GND1
- C26 pad 1: CONTROL_SUPPLY_ADC -> GND3
- C3 pad 1: +5V -> 5v_ISO
- C31 pad 1: GATE_SUPPLY_ADC -> GND2
- C31 pad 2: GND2 -> GND1
- C37 pad 1: Net-(C37-Pad1) -> +15V
- C37 pad 2: Net-(C37-Pad2) -> GND3
- C38 pad 1: Net-(C38-Pad1) -> +5V
- C38 pad 2: Net-(C38-Pad2) -> GND2
- C4 pad 1: +5V -> 5v_ISO
- C40 pad 1: +24V -> +VDC
- C40 pad 2: GND2 -> VBUS -5V
- C41 pad 1: +24V -> +3.3V
- C42 pad 1: Net-(C42-Pad1) -> +5V
- C43 pad 1: +15V -> Net-(C43-Pad1)
- C44 pad 1: Net-(C42-Pad1) -> +VDC
- C44 pad 2: GND2 -> VBUS -5V
- C45 pad 1: +15V -> +3.3V
- C46 pad 1: +3.3V -> +15V
- C46 pad 2: GND2 -> GND3
- C47 pad 1: +3.3V -> +VDC
- C47 pad 2: GND2 -> VBUS -5V
- C48 pad 1: +3.3V -> +VDC
- C48 pad 2: GND2 -> -VDC
- C49 pad 1: +3.3V -> +VDC
- C49 pad 2: GND2 -> -VDC
- C52 pad 1: Net-(C52-Pad1) -> Net-(D16-K)
- C52 pad 2: Net-(C52-Pad2) -> Net-(Q1-DS)
- C53 pad 1: +15V -> Net-(Q1-DS)
- C53 pad 2: Net-(C53-Pad2) -> Net-(D18-A)
- C54 pad 1: Net-(C54-Pad1) -> Net-(D17-K)
- C54 pad 2: Net-(C54-Pad2) -> Net-(Q3-DS)
- C55 pad 1: +15V -> Net-(Q3-DS)
- C55 pad 2: Net-(C55-Pad2) -> Net-(D22-A)
- C56 pad 1: +3.3V -> Net-(D16-K)
- C56 pad 2: GND2 -> Net-(Q1-DS)
- C57 pad 1: Net-(C57-Pad1) -> Net-(Q1-DS)
- C57 pad 2: Net-(C57-Pad2) -> Net-(D18-A)
- C58 pad 1: +15V -> Net-(U10-VDDB)
- C58 pad 2: Net-(C58-Pad2) -> Net-(Q2-DS)
- C59 pad 1: Net-(C52-Pad1) -> Net-(Q2-DS)
- C59 pad 2: Net-(C52-Pad2) -> Net-(U10-GNDB)
- C60 pad 1: +15V -> Net-(U10-VDDB)
- C60 pad 2: Net-(C53-Pad2) -> Net-(Q2-DS)
- C61 pad 1: Net-(C54-Pad1) -> Net-(D17-K)
- C61 pad 2: Net-(C54-Pad2) -> Net-(Q3-DS)
- C62 pad 1: +15V -> Net-(U11-VDDB)
- C62 pad 2: Net-(C55-Pad2) -> Net-(Q4-DS)
- C63 pad 1: Net-(C57-Pad1) -> Net-(Q2-DS)
- C63 pad 2: Net-(C57-Pad2) -> Net-(U10-GNDB)
- C64 pad 1: +15V -> Net-(D19-K)
- C64 pad 2: Net-(C58-Pad2) -> Net-(D19-A)
- C65 pad 1: Net-(C65-Pad1) -> Net-(D19-K)
- C65 pad 2: Net-(C52-Pad2) -> Net-(D19-A)
- C66 pad 2: Net-(C54-Pad2) -> Net-(D20-A)
- C67 pad 1: Net-(C67-Pad1) -> Net-(U12-AINN)
- C67 pad 2: Net-(C57-Pad2) -> Net-(U12-AINP)
- C68 pad 1: Net-(C65-Pad1) -> +3.3V
- C68 pad 2: Net-(C52-Pad2) -> GND2
- C69 pad 2: Net-(C54-Pad2) -> Net-(D20-A)
- C70 pad 1: Net-(C67-Pad1) -> +15V
- C70 pad 2: Net-(C57-Pad2) -> GND3
- C71 pad 1: Net-(C71-Pad1) -> +VDC
- C71 pad 2: Net-(C71-Pad2) -> VBUS -5V
- C73 pad 1: Net-(C73-Pad1) -> +3.3V
- C73 pad 2: Net-(C73-Pad2) -> GND2
- D16 pad 1: Net-(C52-Pad1) -> Net-(D16-K)
- D16 pad 2: Net-(D16-Pad2) -> Net-(D16-A)
- D17 pad 1: Net-(C54-Pad1) -> Net-(D17-K)
- D18 pad 1: Net-(C57-Pad1) -> Net-(D18-K)
- D18 pad 2: Net-(D18-Pad2) -> Net-(D18-A)
- D19 pad 1: Net-(C65-Pad1) -> Net-(D19-K)
- D19 pad 2: Net-(C52-Pad2) -> Net-(D19-A)
- D20 pad 2: Net-(C54-Pad2) -> Net-(D20-A)
- D21 pad 1: Net-(C67-Pad1) -> Net-(D21-K)
- D21 pad 2: Net-(C57-Pad2) -> Net-(D21-A)
- D3 pad 1: GND2 -> Net-(D3-K)
- D4 pad 1: GND2 -> Net-(D4-K)
- D5 pad 1: GND2 -> Net-(D5-K)
- D6 pad 1: GND2 -> Net-(D6-K)
- H4 pad 1: (no net) -> GND
- J5 pad 1: Net-(J5-Pad1) -> U
- J5 pad 2: Net-(J5-Pad2) -> V
- J5 pad 3: Net-(J5-Pad3) -> W
- J6 pad 1: U -> VM
- J6 pad 2: V -> unconnected-(J6-Pin_2-Pad2)
- J6 pad 3: W -> UM
- J7 pad 1: Net-(J7-Pad1) -> +VDC
- J7 pad 2: Net-(J7-Pad2) -> +VDC
- J7 pad 3: Net-(J7-Pad3) -> -VDC
- L1 pad 2: +5V -> 5v_ISO
- L2 pad 1: Net-(C37-Pad2) -> +15V
- L2 pad 2: Net-(C42-Pad1) -> Net-(U11-VDDB)
- L3 pad 1: Net-(C38-Pad2) -> -5V
- L3 pad 2: +15V -> Net-(U11-GNDB)
- L4 pad 1: Net-(C42-Pad1) -> GND3
- L4 pad 2: +3.3V -> Net-(Q4-DS)
- Q1 pad 2: Net-(Q1-Pad2) -> Net-(D19-A)
- Q1 pad 3: Net-(C52-Pad2) -> Net-(Q1-DS)
- Q1 pad 4: Net-(Q1-Pad4) -> Net-(Q1-G)
- Q2 pad 1: Net-(Q1-Pad2) -> Net-(D19-A)
- Q2 pad 3: Net-(C53-Pad2) -> Net-(Q2-DS)
- Q2 pad 4: Net-(Q2-Pad4) -> Net-(Q2-G)
- Q3 pad 2: Net-(Q3-Pad2) -> Net-(D20-A)
- Q3 pad 3: Net-(C54-Pad2) -> Net-(Q3-DS)
- Q4 pad 1: Net-(Q3-Pad2) -> Net-(D20-A)
- Q4 pad 3: Net-(C55-Pad2) -> Net-(Q4-DS)
- Q5 pad 2: Net-(Q5-Pad2) -> Net-(D24-A)
- Q5 pad 3: Net-(C57-Pad2) -> Net-(Q5-DS)
- Q5 pad 4: Net-(Q5-Pad4) -> Net-(Q5-G)
- Q6 pad 1: Net-(Q5-Pad2) -> Net-(D24-A)
- Q6 pad 3: Net-(C58-Pad2) -> Net-(Q6-DS)
- Q6 pad 4: Net-(Q6-Pad4) -> Net-(Q6-G)
- R1 pad 1: Net-(R1-Pad1) -> Net-(U23-A)
- R11 pad 2: LED_1 -> +3.3V
- R12 pad 2: LED_2 -> +3.3V
- R13 pad 2: LED_3 -> +3.3V
- R14 pad 2: LED_4 -> +3.3V
- R2 pad 1: Net-(R2-Pad1) -> Net-(U23-B)
- R25 pad 1: Net-(J5-Pad1) -> UM
- R27 pad 1: Net-(J5-Pad2) -> VM
- R29 pad 1: Net-(J5-Pad3) -> WM
- R3 pad 1: Net-(R3-Pad1) -> Net-(U23-Z)
- R33 pad 1: Net-(C42-Pad1) -> +15V
- R33 pad 2: Net-(R33-Pad2) -> Net-(D16-A)
- R34 pad 1: Net-(R33-Pad2) -> VBUS -5V
- R34 pad 2: GND2 -> Net-(D18-K)
- R35 pad 1: +15V -> Net-(D16-K)
- R35 pad 2: Net-(R35-Pad2) -> Net-(D19-K)
- R36 pad 1: Net-(R35-Pad2) -> Net-(U10-OUTA)
- R36 pad 2: GND2 -> Net-(Q1-G)
- R38 pad 1: Net-(J7-Pad1) -> U
- R4 pad 1: Net-(R4-Pad1) -> Net-(U23-Y)
- R40 pad 1: Net-(J7-Pad2) -> V
- R42 pad 1: Net-(J7-Pad3) -> W
- R47 pad 1: +15V -> Net-(U10-OUTB)
- R47 pad 2: Net-(D16-Pad2) -> Net-(Q2-G)
- R49 pad 1: +15V -> Net-(D19-A)
- R49 pad 2: Net-(D18-Pad2) -> Net-(U12-AINN)
- R5 pad 1: +5V -> 5v_ISO
- R50 pad 1: Net-(C52-Pad1) -> Net-(D19-A)
- R50 pad 2: Net-(C65-Pad1) -> V
- R51 pad 1: Net-(C54-Pad1) -> Net-(D17-K)
- R52 pad 1: Net-(R52-Pad1) -> V
- R52 pad 2: Net-(Q1-Pad4) -> Net-(U12-AINP)
- R53 pad 1: Net-(R53-Pad1) -> +15V
- R53 pad 2: Net-(Q2-Pad4) -> Net-(D21-A)
- R54 pad 1: Net-(R54-Pad1) -> Net-(U11-OUTA)
- R55 pad 1: Net-(R55-Pad1) -> Net-(U11-OUTB)
- R56 pad 1: Net-(C57-Pad1) -> VBUS -5V
- R56 pad 2: Net-(C67-Pad1) -> Net-(D23-K)
- R57 pad 1: Net-(R57-Pad1) -> Net-(D21-K)
- R57 pad 2: Net-(Q5-Pad4) -> Net-(D24-K)
- R58 pad 1: Net-(R58-Pad1) -> Net-(U13-OUTA)
- R58 pad 2: Net-(Q6-Pad4) -> Net-(Q5-G)
- R59 pad 1: Net-(Q1-Pad2) -> Net-(U13-OUTB)
- R59 pad 2: Net-(C71-Pad1) -> Net-(Q6-G)
- R60 pad 1: Net-(Q3-Pad2) -> Net-(D20-A)
- R61 pad 1: Net-(Q1-Pad2) -> Net-(D24-A)
- R61 pad 2: V -> Net-(U15-AINN)
- R62 pad 1: Net-(Q5-Pad2) -> Net-(D24-A)
- R62 pad 2: Net-(C73-Pad1) -> W
- R63 pad 1: Net-(Q3-Pad2) -> Net-(D20-A)
- R64 pad 1: V -> W
- R64 pad 2: Net-(C71-Pad2) -> Net-(U15-AINP)
- R65 pad 1: Net-(Q5-Pad2) -> Net-(D30-A)
- R65 pad 2: W -> STO FBK 24V
- R67 pad 1: W -> SAFE GND
- R67 pad 2: Net-(C73-Pad2) -> Net-(R67-Pad2)
- SW1 pad 1: +3.3V -> GND2
- SW1 pad 2: +3.3V -> GND2
- SW1 pad 3: +3.3V -> GND2
- SW1 pad 4: +3.3V -> GND2
- SW1 pad 5: DIP_4 -> Net-(U1-P04)
- SW1 pad 6: DIP_3 -> Net-(U1-P05)
- SW1 pad 7: DIP_2 -> Net-(U1-P06)
- SW1 pad 8: DIP_1 -> Net-(U1-P07)
- TP1 pad 1: U_CLOCK -> Net-(U22-IN)
- TP10 pad 1: VL -> W_DATA
- TP11 pad 1: UL -> UH
- TP12 pad 1: WL -> UL
- TP13 pad 1: +3.3V -> VH
- TP14 pad 1: V_DATA -> VL
- TP16 pad 1: W_DATA -> WH
- TP2 pad 1: +24V -> +5V
- TP3 pad 1: GND2 -> GND3
- TP4 pad 1: GND2 -> VBUS -5V
- TP5 pad 1: VH -> +15V
- TP6 pad 1: Net-(C42-Pad1) -> -5V
- TP7 pad 1: +15V -> +VDC
- TP8 pad 1: UH -> -VDC
- TP9 pad 1: WH -> V_DATA
- U1 pad 1: RX_ISO -> Net-(U1-~{INT})
- U1 pad 10: +5V -> Net-(U1-P06)
- U1 pad 2: GND1 -> GND2
- U1 pad 3: TX_EN_ISO -> GND2
- U1 pad 4: TX_ISO -> Net-(D3-K)
- U1 pad 5: GND1 -> Net-(D4-K)
- U1 pad 6: Net-(R4-Pad1) -> Net-(D5-K)
- U1 pad 7: Net-(R3-Pad1) -> Net-(D6-K)
- U1 pad 8: Net-(R2-Pad1) -> Net-(U1-P04)
- U1 pad 9: Net-(R1-Pad1) -> Net-(U1-P05)
- U10 pad 3: Net-(C53-Pad2) -> +3.3V
- U10 pad 4: Net-(R53-Pad1) -> GND2
- U10 pad 5: +15V -> STO CH1
- U10 pad 6: Net-(C52-Pad2) -> unconnected-(U10-NC-Pad6)
- U10 pad 7: Net-(R52-Pad1) -> unconnected-(U10-NC-Pad7)
- U10 pad 8: Net-(C52-Pad1) -> +3.3V
- U11 pad 3: Net-(C55-Pad2) -> +3.3V
- U11 pad 4: Net-(R55-Pad1) -> GND2
- U11 pad 5: +15V -> STO CH1
- U11 pad 6: Net-(C54-Pad2) -> unconnected-(U11-NC-Pad6)
- U11 pad 7: Net-(R54-Pad1) -> unconnected-(U11-NC-Pad7)
- U11 pad 8: Net-(C54-Pad1) -> +3.3V
- U12 pad 1: WH -> Net-(D19-K)
- U12 pad 2: WL -> Net-(U12-AINP)
- U12 pad 3: Net-(C58-Pad2) -> Net-(U12-AINN)
- U12 pad 4: Net-(R58-Pad1) -> Net-(D19-A)
- U12 pad 5: +15V -> GND2
- U12 pad 6: Net-(C57-Pad2) -> V_DATA
- U12 pad 7: Net-(R57-Pad1) -> V_CLOCK
- U12 pad 8: Net-(C57-Pad1) -> +3.3V
- U13 pad 1: Net-(C65-Pad1) -> WH
- U13 pad 2: Net-(C71-Pad2) -> WL
- U13 pad 3: Net-(C71-Pad1) -> +3.3V
- U13 pad 4: Net-(C52-Pad2) -> GND2
- U13 pad 5: GND2 -> STO CH1
- U13 pad 6: V_DATA -> unconnected-(U13-NC-Pad6)
- U13 pad 7: U_CLOCK -> unconnected-(U13-NC-Pad7)
- U14 pad 4: Net-(C54-Pad2) -> Net-(D20-A)
- U15 pad 1: Net-(C67-Pad1) -> Net-(D24-K)
- U15 pad 2: Net-(C73-Pad2) -> Net-(U15-AINP)
- U15 pad 3: Net-(C73-Pad1) -> Net-(U15-AINN)
- U15 pad 4: Net-(C57-Pad2) -> Net-(D24-A)
- U15 pad 7: U_CLOCK -> W_CLOCK
- U2 pad 8: +5V -> 5v_ISO
- U3 pad 8: +5V -> 5v_ISO
- U4 pad 8: +5V -> 5v_ISO
- U5 pad 10: LED_3 -> unconnected-(U5B-PC2-Pad10)
- U5 pad 11: LED_4 -> unconnected-(U5B-PC3-Pad11)
- U5 pad 17: UM_ADC -> WM_ADC
- U5 pad 2: LED_2 -> unconnected-(U5B-PC13-Pad2)
- U5 pad 20: VM_ADC -> UM_ADC
- U5 pad 21: WM_ADC -> VM_ADC
- U5 pad 26: CONTROL_SUPPLY_ADC -> unconnected-(U5B-PB0-Pad26)
- U5 pad 29: U_CLOCK -> Net-(U22-IN)
- U5 pad 33: unconnected-(U5-Pad33) -> STO CH2
- U5 pad 51: DIP_4 -> STO EN
- U5 pad 52: DIP_3 -> STO CH1 MCU FBK
- U5 pad 53: DIP_2 -> STO CH2 MCU FBK
- U5 pad 54: DIP_1 -> unconnected-(U5B-PD2-Pad54)
- U5 pad 56: JTRST -> unconnected-(U5B-PB4-Pad56)
- U5 pad 59: unconnected-(U5-Pad59) -> SDA
- U5 pad 61: LED_1 -> SDL
- U7 pad 1: GND1 -> Net-(U7-VIN)
- U7 pad 2: 24V_ISO -> GND1
- U7 pad 5: +24V -> GND2
- U8 pad 1: Net-(C37-Pad1) -> GND2
- U8 pad 6: Net-(C37-Pad2) -> -5V
- U9 pad 1: Net-(C38-Pad1) -> +5V
- U9 pad 3: Net-(R35-Pad2) -> +5V
- U9 pad 4: +24V -> unconnected-(U9-NC-Pad4)
- U9 pad 5: +24V -> +3.3V
Routing:
- net STO CH1: track 0.00 -> 251.1 mm, vias 0 -> 13
- net UM_ADC: track 22.7 -> 206.3 mm
- net VM_ADC: track 29.5 -> 209.4 mm
- net VBUS_ADC: track 27.9 -> 207.2 mm, vias 0 -> 2
- net W_ADC: track 24.2 -> 199.7 mm, vias 0 -> 2
- net V_ADC: track 29.1 -> 200.8 mm, vias 0 -> 2
- net WM_ADC: track 33.2 -> 203.2 mm
- net U_ADC: track 33.8 -> 202.5 mm, vias 0 -> 2
- net VBUS -5V: track 0.00 -> 156.6 mm, vias 0 -> 4
- net STO CH2: track 0.00 -> 137.8 mm, vias 0 -> 4
- net STO EN: track 0.00 -> 129.6 mm, vias 0 -> 6
- net SDA: track 0.00 -> 116.6 mm, vias 0 -> 4
- net -5V: track 0.00 -> 115.0 mm, vias 0 -> 4
- net SDL: track 0.00 -> 114.6 mm, vias 0 -> 4
- net WH: track 44.0 -> 143.1 mm, vias 2 -> 0
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- added copper zone on F.Cu, net +VDC
- added copper zone on F.Cu, net -VDC
- added copper zone on F.Cu, net 5v_ISO
- added copper zone on In1.Cu, net 5v_ISO
- added copper zone on B.Cu, net GND
- added copper zone on In1.Cu, net GND
- added copper zone on In2.Cu, net GND
- added copper zone on In2.Cu, net GND3
- added copper zone on F.Cu, net Net-(D19-A)
- added copper zone on F.Cu, net Net-(D20-A)
- added copper zone on F.Cu, net Net-(D24-A)
- added copper zone on F.Cu, net Net-(Q1-DS)
- added copper zone on F.Cu, net Net-(Q2-DS)
- added copper zone on F.Cu, net Net-(Q3-DS)
- added copper zone on F.Cu, net Net-(Q4-DS)
- added copper zone on F.Cu, net Net-(Q5-DS)
- added copper zone on F.Cu, net Net-(Q6-DS)
- added copper zone on F.Cu, net Net-(U10-OUTA)
- added copper zone on F.Cu, net Net-(U10-OUTB)
- added copper zone on F.Cu, net Net-(U11-OUTA)
- added copper zone on F.Cu, net Net-(U11-OUTB)
- added copper zone on F.Cu, net Net-(U13-OUTA)
- added copper zone on F.Cu, net Net-(U13-OUTB)
- added copper zone on F.Cu, net Net-(U6-SW)
- added copper zone on In2.Cu, net SAFE GND
- added copper zone on F.Cu, net U
- added copper zone on F.Cu, net V
- added copper zone on F.Cu, net W
- removed copper zone on B.Cu, net +15V
- removed copper zone on In1.Cu, net +15V
- removed copper zone on B.Cu, net +24V
- removed copper zone on B.Cu, net +3.3V
- removed copper zone on B.Cu, net +5V
- removed copper zone on In2.Cu, net +5V
- removed copper zone on B.Cu, net 24V_ISO
- removed copper zone on B.Cu, net GND1
- removed copper zone on In1.Cu, net GND1
- removed copper zone on B.Cu, net GND2
- removed copper zone on B.Cu, net Net-(C37-Pad2)
- removed copper zone on B.Cu, net Net-(C38-Pad2)
- removed copper zone on B.Cu, net Net-(C42-Pad1)
- removed copper zone on B.Cu, net Net-(Q1-Pad2)
- removed copper zone on B.Cu, net Net-(Q3-Pad2)
- removed copper zone on B.Cu, net Net-(Q5-Pad2)
- removed copper zone on B.Cu, net Net-(U6-SW)
- removed copper zone on B.Cu, net U
- removed copper zone on B.Cu, net V
- removed copper zone on B.Cu, net W
Other:
- board size 99.8 x 99.3 mm -> 138.4 x 199.6 mm
- board text removed: "+"
- board text removed: "-"
- board text removed: "24V"
- board text removed: "24v"
- board text removed: "3.3v"
- board text removed: "3.3vf"
- board text removed: "BDTMP1"
- board text removed: "CLK"
- board text removed: "DIP1"
- board text removed: "DIP2"
- board text removed: "DIP3"
- board text removed: "DIP4"
- board text removed: "F1"
- board text removed: "F2"
- board text removed: "GATE SUPPLY"
- board text removed: "HSTMP1"
- board text removed: "HSTMP2"
- board text removed: "HVSD 1.0"
- board text removed: "LED1"
- board text removed: "LED2"
- board text removed: "LED3"
- board text removed: "LED4"
- board text removed: "POWER OFF BEFORE SEVICING!"
- board text removed: "PWM"
- board text removed: "TACH"
- board text removed: "UH"
- board text removed: "UL"
- board text removed: "U_DATA"
- board text removed: "VH"
- board text removed: "VL"
- board text removed: "V_DATA"
- board text removed: "WH"
- board text removed: "WL"
- board text removed: "W_DATA"

Commit message: update board layout
Parts:
- added REF**: OSHW-Logo2_14.6x12mm_SilkScreen, Symbol:OSHW-Logo2_14.6x12mm_SilkScreen, F.Cu at (430.8, 234.0)
- added REF**: EO silk 14mm, Library:EO silk 14mm, F.Cu at (416.2, 233.2)
- added REF**: EO silk 3mm, Library:EO silk 3mm, F.Cu at (314.5, 188.8)
- added REF**: OSHW-Logo2_14.6x12mm_SilkScreen, Symbol:OSHW-Logo2_14.6x12mm_SilkScreen, B.Cu at (430.8, 234.0)
- added REF**: EO silk 3mm, Library:EO silk 3mm, B.Cu at (314.5, 188.8)
- added REF**: EO silk 14mm, Library:EO silk 14mm, B.Cu at (416.2, 233.2)
- added TP21: TestPoint, footprints:TestPoint_Pad_3.1x1.6mm, F.Cu at (434.8, 58.0)
- added TP22: TestPoint, footprints:TestPoint_Pad_3.1x1.6mm, F.Cu at (434.8, 54.2)
- C48, C49: moved to B.Cu
- renumbered U5 to U9
Routing:
- net GND2: track 156.9 -> 159.1 mm, vias 53 -> 54
- net +3.3V: track 98.6 -> 100.8 mm, vias 43 -> 44
Other:
- board text added: "+ -"
- board text added: "+15V"
- board text added: "+3.3V"
- board text added: "+5V"
- board text added: "+VDC"
- board text added: "-5V"
- board text added: "-VDC"
- board text added: "1"
- board text added: "2"
- board text added: "24V"
- board text added: "3"
- board text added: "4"
- board text added: "ADC CLK"
- board text added: "G"
- board text added: "GND2"
- board text added: "GND3"
- board text added: "PFC SENSE"
- board text added: "RX+"
- board text added: "RX-"
- board text added: "STO CH1"
- board text added: "STO CH2"
- board text added: "STO EN"
- board text added: "TX+"
- board text added: "TX-"
- board text added: "U DATA"
- board text added: "UH"
- board text added: "UL"
- board text added: "V DATA"
- board text added: "VBUS -5V"
- board text added: "VH"
- board text added: "VL"
- board text added: "W DATA"
- board text added: "WH"
- board text added: "WL"
