File: KiCad/HV servo drive v1/mcu.kicad_sch (KiCad schematic)
At the start: 24 parts, among them J3 PROG, U22 PL133-37TC, U5 STM32F413RGT6, U9 AP2127K-3.3

Commit message: update board layout
Parts:
- added TP1 (x2): TestPoint, footprints:TestPoint_Pad_3.1x1.6mm, symbol Connector:TestPoint
Connections:
- net +3.3V: now also TP1.1
- net GND2: now also TP1.1
