File: KiCad/HV servo drive v1/sto.kicad_sch (KiCad schematic)
At the start: 41 parts, among them J9 Conn_02x03_Top_Bottom, Q8 PMOS, U16 6N137, U17 6N137, U18 FODM217A, U19 FODM217A

Commit message: update board layout
Changed lines of the file:
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@@
   (symbol (lib_id "Device:D_Dual_Series_AKC") (at 82.55 121.92 90) (unit 1)
     (in_bom yes) (on_board yes) (dnp no) (fields_autoplaced)
-    (property "Reference" "D27" (at 80.01 118.8084 90)
-      (effects (font (size 1.27 1.27)) (justify left))
-    )
-    (property "Value" "D_Dual_Series_ACK" (at 80.01 121.3484 90)
+    (property "Reference" "D27" (at 80.01 118.8085 90)
+      (effects (font (size 1.27 1.27)) (justify left))
+    )
+    (property "Value" "D_Dual_Series_ACK" (at 80.01 121.3485 90)
       (effects (font (size 1.27 1.27)) (justify left))
     )
@@
   (symbol (lib_id "Connector:TestPoint") (at 213.36 121.92 0) (unit 1)
     (in_bom yes) (on_board yes) (dnp no) (fields_autoplaced)
-    (property "Reference" "TP23" (at 215.9 117.3479 0)
-      (effects (font (size 1.27 1.27)) (justify left))
-    )
-    (property "Value" "TestPoint" (at 215.9 119.8879 0)
+    (property "Reference" "TP23" (at 215.9 117.348 0)
+      (effects (font (size 1.27 1.27)) (justify left))
+    )
+    (property "Value" "TestPoint" (at 215.9 119.888 0)
       (effects (font (size 1.27 1.27)) (justify left))
     )
@@
   (symbol (lib_id "Device:R") (at 109.22 208.28 90) (unit 1)
     (in_bom yes) (on_board yes) (dnp no) (fields_autoplaced)
-    (property "Reference" "R69" (at 107.95 205.74 0)
-      (effects (font (size 1.27 1.27)) (justify left))
-    )
-    (property "Value" "1K" (at 110.49 205.74 0)
-      (effects (font (size 1.27 1.27)) (justify left))
+    (property "Reference" "R69" (at 109.22 201.93 90)
+      (effects (font (size 1.27 1.27)))
+    )
+    (property "Value" "1K" (at 109.22 204.47 90)
+      (effects (font (size 1.27 1.27)))
     )
     (property "Footprint" "Resistor_SMD:R_0603_1608Metric" (at 109.22 210.058 90)
@@
   (symbol (lib_id "Connector:TestPoint") (at 213.36 113.03 0) (unit 1)
     (in_bom yes) (on_board yes) (dnp no) (fields_autoplaced)
-    (property "Reference" "TP22" (at 215.9 108.4579 0)
-      (effects (font (size 1.27 1.27)) (justify left))
-    )
-    (property "Value" "TestPoint" (at 215.9 110.9979 0)
+    (property "Reference" "TP22" (at 215.9 108.458 0)
+      (effects (font (size 1.27 1.27)) (justify left))
+    )
+    (property "Value" "TestPoint" (at 215.9 110.998 0)
       (effects (font (size 1.27 1.27)) (justify left))
     )
@@
   (symbol (lib_id "Device:C") (at 91.44 142.24 0) (unit 1)
     (in_bom yes) (on_board yes) (dnp no) (fields_autoplaced)
-    (property "Reference" "C98" (at 95.25 140.9699 0)
-      (effects (font (size 1.27 1.27)) (justify left))
-    )
-    (property "Value" "10uf" (at 95.25 143.5099 0)
+    (property "Reference" "C98" (at 95.25 140.97 0)
+      (effects (font (size 1.27 1.27)) (justify left))
+    )
+    (property "Value" "10uf" (at 95.25 143.51 0)
       (effects (font (size 1.27 1.27)) (justify left))
     )
@@
   (symbol (lib_id "Device:R") (at 101.6 208.28 90) (unit 1)
     (in_bom yes) (on_board yes) (dnp no) (fields_autoplaced)
-    (property "Reference" "R67" (at 100.33 205.74 0)
-      (effects (font (size 1.27 1.27)) (justify left))
-    )
-    (property "Value" "1K" (at 102.87 205.74 0)
-      (effects (font (size 1.27 1.27)) (justify left))
+    (property "Reference" "R67" (at 101.6 201.93 90)
+      (effects (font (size 1.27 1.27)))
+    )
+    (property "Value" "1K" (at 101.6 204.47 90)
+      (effects (font (size 1.27 1.27)))
     )
     (property "Footprint" "Resistor_SMD:R_0603_1608Metric" (at 101.6 210.058 90)
@@
   (symbol (lib_id "Device:C") (at 168.91 148.59 0) (unit 1)
     (in_bom yes) (on_board yes) (dnp no) (fields_autoplaced)
-    (property "Reference" "C99" (at 172.72 147.3199 0)
-      (effects (font (size 1.27 1.27)) (justify left))
-    )
-    (property "Value" "0.1uf" (at 172.72 149.8599 0)
+    (property "Reference" "C99" (at 172.72 147.32 0)
+      (effects (font (size 1.27 1.27)) (justify left))
+    )
+    (property "Value" "0.1uf" (at 172.72 149.86 0)
       (effects (font (size 1.27 1.27)) (justify left))
     )
@@
   (symbol (lib_id "Device:D_Dual_Series_AKC") (at 73.66 200.66 90) (unit 1)
     (in_bom yes) (on_board yes) (dnp no) (fields_autoplaced)
-    (property "Reference" "D29" (at 71.12 197.5484 90)
-      (effects (font (size 1.27 1.27)) (justify left))
-    )
-    (property "Value" "D_Dual_Series_ACK" (at 71.12 200.0884 90)
+    (property "Reference" "D29" (at 71.12 197.5485 90)
+      (effects (font (size 1.27 1.27)) (justify left))
+    )
+    (property "Value" "D_Dual_Series_ACK" (at 71.12 200.0885 90)
       (effects (font (size 1.27 1.27)) (justify left))
     )
@@
   )
   (symbol (lib_id "Device:D_Zener") (at 101.6 142.24 270) (unit 1)
-    (in_bom yes) (on_board yes) (dnp no)
+    (in_bom yes) (on_board yes) (dnp no) (fields_autoplaced)
     (property "Reference" "D28" (at 104.14 140.97 90)
       (effects (font (size 1.27 1.27)) (justify left))
     )
-    (property "Value" "BZT52C5V1" (at 102.87 143.51 90)
+    (property "Value" "BZT52C5V1" (at 104.14 143.51 90)
       (effects (font (size 1.27 1.27)) (justify left))
     )
@@
   )
   (symbol (lib_id "Isolator:FODM217A") (at 138.43 201.93 0) (mirror y) (unit 1)
-    (in_bom yes) (on_board yes) (dnp no)
+    (in_bom yes) (on_board yes) (dnp no) (fields_autoplaced)
     (property "Reference" "U19" (at 138.43 193.04 0)
       (effects (font (size 1.27 1.27)))
@@
   )
   (symbol (lib_id "Isolator:FODM217A") (at 138.43 186.69 0) (mirror y) (unit 1)
-    (in_bom yes) (on_board yes) (dnp no)
+    (in_bom yes) (on_board yes) (dnp no) (fields_autoplaced)
     (property "Reference" "U18" (at 138.43 177.8 0)
       (effects (font (size 1.27 1.27)))
@@
   (symbol (lib_id "Device:C") (at 168.91 93.98 0) (unit 1)
     (in_bom yes) (on_board yes) (dnp no) (fields_autoplaced)
-    (property "Reference" "C96" (at 172.72 92.7099 0)
-      (effects (font (size 1.27 1.27)) (justify left))
-    )
-    (property "Value" "0.1uf" (at 172.72 95.2499 0)
+    (property "Reference" "C96" (at 172.72 92.71 0)
+      (effects (font (size 1.27 1.27)) (justify left))
+    )
+    (property "Value" "0.1uf" (at 172.72 95.25 0)
       (effects (font (size 1.27 1.27)) (justify left))
     )
@@
   (symbol (lib_id "Connector:TestPoint") (at 213.36 130.81 0) (unit 1)
     (in_bom yes) (on_board yes) (dnp no) (fields_autoplaced)
-    (property "Reference" "TP24" (at 215.9 126.2379 0)
-      (effects (font (size 1.27 1.27)) (justify left))
-    )
-    (property "Value" "TestPoint" (at 215.9 128.7779 0)
+    (property "Reference" "TP24" (at 215.9 126.238 0)
+      (effects (font (size 1.27 1.27)) (justify left))
+    )
+    (property "Value" "TestPoint" (at 215.9 128.778 0)
       (effects (font (size 1.27 1.27)) (justify left))
     )
@@
   (symbol (lib_id "Device:C") (at 91.44 87.63 0) (unit 1)
     (in_bom yes) (on_board yes) (dnp no) (fields_autoplaced)
-    (property "Reference" "C97" (at 95.25 86.3599 0)
-      (effects (font (size 1.27 1.27)) (justify left))
-    )
-    (property "Value" "10uf" (at 95.25 88.8999 0)
+    (property "Reference" "C97" (at 95.25 86.36 0)
+      (effects (font (size 1.27 1.27)) (justify left))
+    )
+    (property "Value" "10uf" (at 95.25 88.9 0)
       (effects (font (size 1.27 1.27)) (justify left))
     )
@@
   )
   (symbol (lib_id "Device:D_Zener") (at 101.6 87.63 270) (unit 1)
-    (in_bom yes) (on_board yes) (dnp no)
+    (in_bom yes) (on_board yes) (dnp no) (fields_autoplaced)
     (property "Reference" "D25" (at 104.14 86.36 90)
       (effects (font (size 1.27 1.27)) (justify left))
     )
-    (property "Value" "BZT52C5V1" (at 102.87 88.9 90)
+    (property "Value" "BZT52C5V1" (at 104.14 88.9 90)
       (effects (font (size 1.27 1.27)) (justify left))
     )
@@
   (symbol (lib_id "Device:D_Dual_Series_AKC") (at 83.82 68.58 90) (unit 1)
     (in_bom yes) (on_board yes) (dnp no) (fields_autoplaced)
-    (property "Reference" "D26" (at 81.28 65.4684 90)
-      (effects (font (size 1.27 1.27)) (justify left))
-    )
-    (property "Value" "D_Dual_Series_ACK" (at 81.28 68.0084 90)
-      (effects (font (size 1.27 1.27)) (justify left))
-    )
+    (property "Reference" "D26" (at 81.28 65.4685 90)
+      (effects (font (size 1.27 1.27)) (justify left))
+    )
+    (property "Value" "D_Dual_Series_ACK" (at 81.28 68.0085 90)
+      (effects (font (size 1.27 1.27)) (justify left))
+    )
